File: _saved_file58C423FA.sch (KiCad schematic (older format))
At the start: 52 parts, among them P3 Servo In/Ext. Mod, P4 Output/Monitor, U6 OPA4227, U7 OPA2227, U8 8DIP, U9 8DIP

Commit message: Board connectors placed
Parts:
- S7: footprint footprints:SPDT-Horizontal -> footprints:CJS-1200TB-SPDT
Changed lines of the file:
@@
 F 0 "S7" V 8250 4300 60  0000 C CNN
 F 1 "spdt" H 8100 4700 60  0000 C CNN
-F 2 "footprints:SPDT-Horizontal" H 8100 4450 60  0001 C CNN
+F 2 "footprints:CJS-1200TB-SPDT" H 8100 4450 60  0001 C CNN
 F 3 "" H 8100 4450 60  0000 C CNN
 	1    8100 4450
