File: file58C3664B.sch (KiCad schematic (older format))
At the start: 10 parts

Commit message: Schematic complete
Parts:
- gave numbers to parts that had none: 10
Changed lines of the file:
@@
 LIBS:valves
 LIBS:all_components
+LIBS:mini_pid-cache
 EELAYER 25 0
 EELAYER END
@@
 $EndComp
 $Comp
-L C C?
+L C C1
 U 1 1 58C3823D
 P 2900 1500
-F 0 "C?" H 2925 1600 50  0000 L CNN
+F 0 "C1" H 2925 1600 50  0000 L CNN
 F 1 "10uF" H 2925 1400 50  0000 L CNN
 F 2 "Capacitors_SMD:C_0603_HandSoldering" H 2938 1350 50  0001 C CNN
@@
 $EndComp
 $Comp
-L C C?
+L C C2
 U 1 1 58C38244
 P 2900 1900
-F 0 "C?" H 2925 2000 50  0000 L CNN
+F 0 "C2" H 2925 2000 50  0000 L CNN
 F 1 "10uF" H 2925 1800 50  0000 L CNN
 F 2 "Capacitors_SMD:C_0603_HandSoldering" H 2938 1750 50  0001 C CNN
@@
 $EndComp
 $Comp
-L -15V #PWR?
+L -15V #PWR4
 U 1 1 58C3824B
 P 3500 2150
-F 0 "#PWR?" H 3500 2250 50  0001 C CNN
+F 0 "#PWR4" H 3500 2250 50  0001 C CNN
 F 1 "-15V" H 3500 2300 50  0000 C CNN
 F 2 "" H 3500 2150 50  0000 C CNN
@@
 $EndComp
 $Comp
-L ED2610 U?
+L ED2610 U1
 U 1 1 58C38257
 P 2250 1700
-F 0 "U?" H 2250 1600 60  0000 C CNN
+F 0 "U1" H 2250 1600 60  0000 C CNN
 F 1 "ED2610" H 2250 1500 60  0000 C CNN
 F 2 "footprints:ED2610" H 2250 1700 60  0001 C CNN
@@
 $EndComp
 $Comp
-L C C?
+L C C4
 U 1 1 58C38264
 P 3500 1500
-F 0 "C?" H 3525 1600 50  0000 L CNN
+F 0 "C4" H 3525 1600 50  0000 L CNN
 F 1 "0.1uF" H 3525 1400 50  0000 L CNN
 F 2 "Capacitors_SMD:C_0603_HandSoldering" H 3538 1350 50  0001 C CNN
@@
 $EndComp
 $Comp
-L C C?
+L C C5
 U 1 1 58C3826B
 P 3500 1900
-F 0 "C?" H 3525 2000 50  0000 L CNN
+F 0 "C5" H 3525 2000 50  0000 L CNN
 F 1 "0.1uF" H 3525 1800 50  0000 L CNN
 F 2 "Capacitors_SMD:C_0603_HandSoldering" H 3538 1750 50  0001 C CNN
@@
 $EndComp
 $Comp
-L C C?
+L C C3
 U 1 1 58C38272
 P 3250 1700
-F 0 "C?" H 3275 1800 50  0000 L CNN
+F 0 "C3" H 3275 1800 50  0000 L CNN
 F 1 "0.1uF" H 3275 1600 50  0000 L CNN
 F 2 "Capacitors_SMD:C_0603_HandSoldering" H 3288 1550 50  0001 C CNN
@@
 Connection ~ 3500 1300
 $Comp
-L DB9 J?
+L DB9 J1
 U 1 1 58C38477
 P 1100 1750
-F 0 "J?" H 1100 2300 50  0000 C CNN
+F 0 "J1" H 1100 2300 50  0000 C CNN
 F 1 "DB9" H 1100 1200 50  0000 C CNN
 F 2 "" H 1100 1750 50  0000 C CNN
@@
 $EndComp
 $Comp
-L TL4050B51 D?
+L TL4050B51 D1
 U 1 1 58C39DF1
 P 4250 1750
-F 0 "D?" H 4250 1850 50  0000 C CNN
+F 0 "D1" H 4250 1850 50  0000 C CNN
 F 1 "TL4050B51" H 4250 1650 50  0000 C CNN
 F 2 "TO_SOT_Packages_SMD:SOT-23" H 4250 1750 50  0001 C CNN
@@
 $EndComp
 $Comp
-L R R?
+L R R1
 U 1 1 58C39DF8
 P 4250 1300
-F 0 "R?" V 4330 1300 50  0000 C CNN
+F 0 "R1" V 4330 1300 50  0000 C CNN
 F 1 "333" V 4250 1300 50  0000 C CNN
 F 2 "Resistors_SMD:R_0603_HandSoldering" V 4180 1300 50  0001 C CNN
@@
 $EndComp
 $Comp
-L TL4050B51 D?
+L TL4050B51 D2
 U 1 1 58C39E0B
 P 4250 2200
-F 0 "D?" H 4250 2300 50  0000 C CNN
+F 0 "D2" H 4250 2300 50  0000 C CNN
 F 1 "TL4050B51" H 4250 2100 50  0000 C CNN
 F 2 "TO_SOT_Packages_SMD:SOT-23" H 4250 2200 50  0001 C CNN

Commit message: Made both circiuts identical
Parts:
- removed D1, D2: TL4050B51, TO_SOT_Packages_SMD:SOT-23, symbol TL4050B51
- removed R1: 333, Resistors_SMD:R_0603_HandSoldering, symbol R
- C1, C2, C3, C4, C5: footprint Capacitors_SMD:C_0603_HandSoldering -> (none)
- U1: footprint footprints:ED2610 -> (none)
Changed lines of the file:
@@
 F 0 "C1" H 2925 1600 50  0000 L CNN
 F 1 "10uF" H 2925 1400 50  0000 L CNN
-F 2 "Capacitors_SMD:C_0603_HandSoldering" H 2938 1350 50  0001 C CNN
+F 2 "" H 2938 1350 50  0001 C CNN
 F 3 "" H 2900 1500 50  0000 C CNN
 	1    2900 1500
@@
 F 0 "C2" H 2925 2000 50  0000 L CNN
 F 1 "10uF" H 2925 1800 50  0000 L CNN
-F 2 "Capacitors_SMD:C_0603_HandSoldering" H 2938 1750 50  0001 C CNN
+F 2 "" H 2938 1750 50  0001 C CNN
 F 3 "" H 2900 1900 50  0000 C CNN
 	1    2900 1900
@@
 F 0 "U1" H 2250 1600 60  0000 C CNN
 F 1 "ED2610" H 2250 1500 60  0000 C CNN
-F 2 "footprints:ED2610" H 2250 1700 60  0001 C CNN
+F 2 "" H 2250 1700 60  0001 C CNN
 F 3 "" H 2250 1700 60  0000 C CNN
 	1    2250 1700
@@
 F 0 "C4" H 3525 1600 50  0000 L CNN
 F 1 "0.1uF" H 3525 1400 50  0000 L CNN
-F 2 "Capacitors_SMD:C_0603_HandSoldering" H 3538 1350 50  0001 C CNN
+F 2 "" H 3538 1350 50  0001 C CNN
 F 3 "" H 3500 1500 50  0000 C CNN
 	1    3500 1500
@@
 F 0 "C5" H 3525 2000 50  0000 L CNN
 F 1 "0.1uF" H 3525 1800 50  0000 L CNN
-F 2 "Capacitors_SMD:C_0603_HandSoldering" H 3538 1750 50  0001 C CNN
+F 2 "" H 3538 1750 50  0001 C CNN
 F 3 "" H 3500 1900 50  0000 C CNN
 	1    3500 1900
@@
 F 0 "C3" H 3275 1800 50  0000 L CNN
 F 1 "0.1uF" H 3275 1600 50  0000 L CNN
-F 2 "Capacitors_SMD:C_0603_HandSoldering" H 3288 1550 50  0001 C CNN
+F 2 "" H 3288 1550 50  0001 C CNN
 F 3 "" H 3250 1700 50  0000 C CNN
 	1    3250 1700
@@
 F 0 "J1" H 1100 2300 50  0000 C CNN
 F 1 "DB9" H 1100 1200 50  0000 C CNN
-F 2 "" H 1100 1750 50  0000 C CNN
+F 2 "" H 1100 1750 50  0001 C CNN
 F 3 "" H 1100 1750 50  0000 C CNN
 	1    1100 1750
@@
 Wire Wire Line
 	1850 1300 3500 1300
-$Comp
-L +15V #PWR07
-U 1 1 58C39DEB
-P 4250 1100
-F 0 "#PWR07" H 4250 950 50  0001 C CNN
-F 1 "+15V" H 4250 1240 50  0000 C CNN
-F 2 "" H 4250 1100 50  0000 C CNN
-F 3 "" H 4250 1100 50  0000 C CNN
-	1    4250 1100
-	1    0    0    -1
-$EndComp
-$Comp
-L TL4050B51 D1
-U 1 1 58C39DF1
-P 4250 1750
-F 0 "D1" H 4250 1850 50  0000 C CNN
-F 1 "TL4050B51" H 4250 1650 50  0000 C CNN
-F 2 "TO_SOT_Packages_SMD:SOT-23" H 4250 1750 50  0001 C CNN
-F 3 "" H 4250 1750 50  0000 C CNN
-	1    4250 1750
-	0    1    1    0
-$EndComp
-$Comp
-L R R1
-U 1 1 58C39DF8
-P 4250 1300
-F 0 "R1" V 4330 1300 50  0000 C CNN
-F 1 "333" V 4250 1300 50  0000 C CNN
-F 2 "Resistors_SMD:R_0603_HandSoldering" V 4180 1300 50  0001 C CNN
-F 3 "" H 4250 1300 50  0000 C CNN
-	1    4250 1300
-	1    0    0    -1
-$EndComp
-Text Label 4700 1500 0    60   ~ 0
-10V
-Wire Wire Line
-	4250 1100 4250 1150
-Wire Wire Line
-	4250 1450 4250 1550
-Wire Wire Line
-	4250 1950 4250 2000
-Wire Wire Line
-	4250 1500 4700 1500
-Connection ~ 4250 1500
-$Comp
-L GND #PWR08
-U 1 1 58C39E05
-P 4250 2450
-F 0 "#PWR08" H 4250 2200 50  0001 C CNN
-F 1 "GND" H 4250 2300 50  0000 C CNN
-F 2 "" H 4250 2450 50  0000 C CNN
-F 3 "" H 4250 2450 50  0000 C CNN
-	1    4250 2450
-	1    0    0    -1
-$EndComp
-$Comp
-L TL4050B51 D2
-U 1 1 58C39E0B
-P 4250 2200
-F 0 "D2" H 4250 2300 50  0000 C CNN
-F 1 "TL4050B51" H 4250 2100 50  0000 C CNN
-F 2 "TO_SOT_Packages_SMD:SOT-23" H 4250 2200 50  0001 C CNN
-F 3 "" H 4250 2200 50  0000 C CNN
-	1    4250 2200
-	0    1    1    0
-$EndComp
-Wire Wire Line
-	4250 2400 4250 2450
 $EndSCHEMATC

Commit message: Board connectors placed
Parts:
- C1, C2, C3, C4, C5: footprint (none) -> Capacitors_SMD:C_0805_HandSoldering
- J1: footprint (none) -> footprints:DB9_Throughhole
- U1: footprint (none) -> footprints:ED2610
Changed lines of the file:
@@
 $EndDescr
 $Comp
-L +15V #PWR3
+L +15V #PWR01
 U 1 1 58C38237
 P 3500 1300
-F 0 "#PWR3" H 3500 1150 50  0001 C CNN
+F 0 "#PWR01" H 3500 1150 50  0001 C CNN
 F 1 "+15V" H 3500 1440 50  0000 C CNN
 F 2 "" H 3500 1300 50  0000 C CNN
@@
 F 0 "C1" H 2925 1600 50  0000 L CNN
 F 1 "10uF" H 2925 1400 50  0000 L CNN
-F 2 "" H 2938 1350 50  0001 C CNN
+F 2 "Capacitors_SMD:C_0805_HandSoldering" H 2938 1350 50  0001 C CNN
 F 3 "" H 2900 1500 50  0000 C CNN
 	1    2900 1500
@@
 F 0 "C2" H 2925 2000 50  0000 L CNN
 F 1 "10uF" H 2925 1800 50  0000 L CNN
-F 2 "" H 2938 1750 50  0001 C CNN
+F 2 "Capacitors_SMD:C_0805_HandSoldering" H 2938 1750 50  0001 C CNN
 F 3 "" H 2900 1900 50  0000 C CNN
 	1    2900 1900
@@
 $EndComp
 $Comp
-L PWR_FLAG #FLG3
+L PWR_FLAG #FLG02
 U 1 1 58C38251
 P 2900 1250
-F 0 "#FLG3" H 2900 1345 50  0001 C CNN
+F 0 "#FLG02" H 2900 1345 50  0001 C CNN
 F 1 "PWR_FLAG" H 2900 1430 50  0000 C CNN
 F 2 "" H 2900 1250 50  0000 C CNN
@@
 F 0 "U1" H 2250 1600 60  0000 C CNN
 F 1 "ED2610" H 2250 1500 60  0000 C CNN
-F 2 "" H 2250 1700 60  0001 C CNN
+F 2 "footprints:ED2610" H 2250 1700 60  0001 C CNN
 F 3 "" H 2250 1700 60  0000 C CNN
 	1    2250 1700
@@
 $EndComp
 $Comp
-L GND #PWR2
+L GND #PWR03
 U 1 1 58C3825E
 P 2650 1700
-F 0 "#PWR2" H 2650 1450 50  0001 C CNN
+F 0 "#PWR03" H 2650 1450 50  0001 C CNN
 F 1 "GND" H 2650 1550 50  0000 C CNN
 F 2 "" H 2650 1700 50  0000 C CNN
@@
 F 0 "C4" H 3525 1600 50  0000 L CNN
 F 1 "0.1uF" H 3525 1400 50  0000 L CNN
-F 2 "" H 3538 1350 50  0001 C CNN
+F 2 "Capacitors_SMD:C_0805_HandSoldering" H 3538 1350 50  0001 C CNN
 F 3 "" H 3500 1500 50  0000 C CNN
 	1    3500 1500
@@
 F 0 "C5" H 3525 2000 50  0000 L CNN
 F 1 "0.1uF" H 3525 1800 50  0000 L CNN
-F 2 "" H 3538 1750 50  0001 C CNN
+F 2 "Capacitors_SMD:C_0805_HandSoldering" H 3538 1750 50  0001 C CNN
 F 3 "" H 3500 1900 50  0000 C CNN
 	1    3500 1900
@@
 F 0 "C3" H 3275 1800 50  0000 L CNN
 F 1 "0.1uF" H 3275 1600 50  0000 L CNN
-F 2 "" H 3288 1550 50  0001 C CNN
+F 2 "Capacitors_SMD:C_0805_HandSoldering" H 3288 1550 50  0001 C CNN
 F 3 "" H 3250 1700 50  0000 C CNN
 	1    3250 1700
@@
 $EndComp
 $Comp
-L PWR_FLAG #FLG2
+L PWR_FLAG #FLG04
 U 1 1 58C38279
 P 2650 1600
-F 0 "#FLG2" H 2650 1695 50  0001 C CNN
+F 0 "#FLG04" H 2650 1695 50  0001 C CNN
 F 1 "PWR_FLAG" H 2650 1780 50  0000 C CNN
 F 2 "" H 2650 1600 50  0000 C CNN
@@
 $EndComp
 $Comp
-L PWR_FLAG #FLG1
+L PWR_FLAG #FLG05
 U 1 1 58C3827F
 P 2300 2250
-F 0 "#FLG1" H 2300 2345 50  0001 C CNN
+F 0 "#FLG05" H 2300 2345 50  0001 C CNN
 F 1 "PWR_FLAG" H 2300 2430 50  0000 C CNN
 F 2 "" H 2300 2250 50  0000 C CNN
@@
 F 0 "J1" H 1100 2300 50  0000 C CNN
 F 1 "DB9" H 1100 1200 50  0000 C CNN
-F 2 "" H 1100 1750 50  0001 C CNN
+F 2 "footprints:DB9_Throughhole" H 1100 1750 50  0001 C CNN
 F 3 "" H 1100 1750 50  0000 C CNN
 	1    1100 1750
@@
 	1600 2150 1550 2150
 $Comp
-L GND #PWR1
+L GND #PWR06
 U 1 1 58C385D7
 P 1600 2250
-F 0 "#PWR1" H 1600 2000 50  0001 C CNN
+F 0 "#PWR06" H 1600 2000 50  0001 C CNN
 F 1 "GND" H 1600 2100 50  0000 C CNN
 F 2 "" H 1600 2250 50  0000 C CNN
