File: file58C423FA.sch (KiCad schematic (older format))
At the start: 52 parts, among them P3 Servo In/Ext. Mod, P4 Output/Monitor, U6 OPA4227, U7 OPA2227, U8 8DIP, U9 8DIP

Commit message: PI circuit 1 done
Parts:
- S7: footprint footprints:SPDT-Horizontal -> footprints:CJS-1200TB-SPDT
Connections:
- net -5V: no longer C34.2, C35.2
- net GND: now also C34.2, C35.2
- net set_point: no longer R28.2, R29.1, S5.3, U6.1
- new net set_point_mon: R28.2, R29.1, S5.3, U6.1

Commit message: Track routing done.
Parts:
- RV4, RV5, RV6: symbol POT -> POT-RESCUE-mini_pid
Changed lines of the file:
@@
 EESchema Schematic File Version 2
+LIBS:mini_pid-rescue
 LIBS:power
 LIBS:device
@@
 $EndComp
 $Comp
-L POT RV6
+L POT-RESCUE-mini_pid RV6
 U 1 1 58C93987
 P 7500 2600
+AR Path="/58C93987" Ref="RV6"  Part="1"
+AR Path="/58C423FB/58C93987" Ref="RV6"  Part="1"
 F 0 "RV6" H 7500 2500 50  0000 C CNN
 F 1 "10k" H 7500 2600 50  0000 C CNN
@@
 set_point_mon
 $Comp
-L POT RV5
+L POT-RESCUE-mini_pid RV5
 U 1 1 58C93A96
 P 5000 5000
+AR Path="/58C93A96" Ref="RV5"  Part="1"
+AR Path="/58C423FB/58C93A96" Ref="RV5"  Part="1"
 F 0 "RV5" H 5000 4900 50  0000 C CNN
 F 1 "1k" H 5000 5000 50  0000 C CNN
@@
 $EndComp
 $Comp
-L POT RV4
+L POT-RESCUE-mini_pid RV4
 U 1 1 58C93AAC
 P 2000 1950
+AR Path="/58C93AAC" Ref="RV4"  Part="1"
+AR Path="/58C423FB/58C93AAC" Ref="RV4"  Part="1"
 F 0 "RV4" H 2000 1850 50  0000 C CNN
 F 1 "1k" H 2000 1950 50  0000 C CNN
