File: mini_pid.kicad_pcb (KiCad board)
At the start: 2 copper layers, 329.6 x 208.1 mm, 111 parts, among them J1 DB9, P1 Servo In/Ext. Mod, P2 Output/Monitor, P3 Servo In/Ext. Mod, P4 Output/Monitor, U1 ED2610, U2 OPA4227, U3 OPA2227, U4 8DIP, U5 8DIP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

Commit message: Interactive routing FTW. PI circuit 1 done.
Parts:
- added REF**: Via-0.6mm, footprints:Via-0.6mm, F.Cu at (58.0, 124.8)
- added REF**: Via-0.6mm, footprints:Via-0.6mm, F.Cu at (120.2, 136.8)
- added REF**: Via-0.6mm, footprints:Via-0.6mm, F.Cu at (122.3, 136.8)
- added REF**: Via-0.6mm, footprints:Via-0.6mm, F.Cu at (125.4, 136.7)
- added REF**: Via-0.6mm, footprints:Via-0.6mm, F.Cu at (140.8, 156.6)
- added REF**: Via-0.6mm, footprints:Via-0.6mm, F.Cu at (140.9, 161.3)
- added REF**: Via-0.6mm, footprints:Via-0.6mm, F.Cu at (129.3, 162.6)
- added REF**: Via-0.6mm, footprints:Via-0.6mm, F.Cu at (118.4, 159.9)
- added REF**: Via-0.6mm, footprints:Via-0.6mm, F.Cu at (123.9, 160.0)
- added REF**: Via-0.6mm, footprints:Via-0.6mm, F.Cu at (129.3, 129.6)
- added REF**: Via-0.6mm, footprints:Via-0.6mm, F.Cu at (126.8, 128.3)
- added REF**: Via-0.6mm, footprints:Via-0.6mm, F.Cu at (58.1, 120.2)
- added REF**: Via-0.6mm, footprints:Via-0.6mm, F.Cu at (50.1, 139.0)
- added REF**: Via-0.6mm, footprints:Via-0.6mm, F.Cu at (45.1, 132.7)
- added REF**: Via-0.6mm, footprints:Via-0.6mm, F.Cu at (47.1, 132.7)
- added REF**: Via-0.6mm, footprints:Via-0.6mm, F.Cu at (54.0, 130.1)
- added REF**: Via-0.6mm, footprints:Via-0.6mm, F.Cu at (51.6, 128.8)
- added REF**: Via-0.6mm, footprints:Via-0.6mm, F.Cu at (65.4, 159.7)
- added REF**: Via-0.6mm, footprints:Via-0.6mm, F.Cu at (65.5, 162.6)
- added REF**: Via-0.6mm, footprints:Via-0.6mm, F.Cu at (57.1, 163.6)
- added REF**: Via-0.6mm, footprints:Via-0.6mm, F.Cu at (40.6, 163.4)
- added REF**: Via-0.6mm, footprints:Via-0.6mm, F.Cu at (43.2, 160.6)
- added REF**: Via-0.6mm, footprints:Via-0.6mm, F.Cu at (58.1, 121.4)
- added REF**: Via-0.6mm, footprints:Via-0.6mm, F.Cu at (48.1, 160.8)
- added REF**: Via-0.6mm, footprints:Via-0.6mm, F.Cu at (159.2, 77.0)
- added REF**: Via-0.6mm, footprints:Via-0.6mm, F.Cu at (161.3, 70.6)
- added REF**: Via-0.6mm, footprints:Via-0.6mm, F.Cu at (157.0, 70.6)
- added REF**: Via-0.6mm, footprints:Via-0.6mm, F.Cu at (58.0, 186.1)
- added REF**: Via-0.6mm, footprints:Via-0.6mm, F.Cu at (58.5, 188.1)
- added REF**: Via-0.6mm, footprints:Via-0.6mm, F.Cu at (118.2, 164.2)
- added REF**: Via-0.6mm, footprints:Via-0.6mm, F.Cu at (132.0, 187.6)
- added REF**: Via-0.6mm, footprints:Via-0.6mm, F.Cu at (114.5, 182.4)
- added REF**: Via-0.6mm, footprints:Via-0.6mm, F.Cu at (121.6, 183.1)
- moved D4 8.89 mm to (123.1, 180.5)
- moved R24 8.62 mm to (122.4, 186.7), turned to 0 degrees
- moved R23 7.88 mm to (113.5, 186.6)
- moved D3 7.52 mm to (113.5, 180.0)
- moved U4 5.12 mm to (43.5, 96.0)
- moved R10 4.09 mm to (59.7, 106.1)
- moved R11 4.09 mm to (59.7, 111.2)
- moved R8 4.09 mm to (59.7, 96.0)
- moved R9 4.09 mm to (59.7, 101.1)
- moved R12 4.09 mm to (65.6, 98.5)
- moved R13 4.09 mm to (65.6, 103.6)
- moved R14 4.09 mm to (65.6, 108.7)
- moved R15 4.09 mm to (65.6, 113.8)
- moved R31 3.89 mm to (134.9, 102.1)
- moved R32 3.89 mm to (134.8, 107.2)
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Routing:
- net +15V: track 0.00 -> 437.6 mm, vias 0 -> 10
- net -15V: track 0.00 -> 397.4 mm, vias 0 -> 8
- net Net-(P1-Pad1): track 0.00 -> 142.2 mm, vias 0 -> 1
- net Net-(C12-Pad1): track 0.00 -> 141.4 mm, vias 0 -> 1
- net Net-(P2-Pad3): track 0.00 -> 105.6 mm, vias 0 -> 1
- net Net-(R16-Pad2): track 0.00 -> 104.8 mm, vias 0 -> 2
- net Net-(P1-Pad3): track 0.00 -> 100.7 mm, vias 0 -> 1
- net /PI Circuit 1/+5V: track 0.00 -> 94.3 mm, vias 0 -> 1
- net Net-(R21-Pad2): track 0.00 -> 91.1 mm, vias 0 -> 2
- net /PI Circuit 1/set_point_mon: track 0.00 -> 82.3 mm, vias 0 -> 2
- net Net-(C19-Pad1): track 0.00 -> 70.7 mm
- net /PI Circuit 1/-5V: track 0.00 -> 69.7 mm, vias 0 -> 1
- net Net-(R16-Pad1): track 0.00 -> 69.3 mm, vias 0 -> 2
- net Net-(R10-Pad2): track 0.00 -> 68.5 mm
- net Net-(R20-Pad1): track 0.00 -> 56.7 mm, vias 0 -> 2
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Other:
- net class Power: clearance 0.4 -> 0.381

Commit message: Gerber and drill files created.
Parts:
- added REF**: Via-0.6mm, footprints:Via-0.6mm, F.Cu at (132.6, 162.6)
- added REF**: Via-0.6mm, footprints:Via-0.6mm, F.Cu at (127.2, 160.8)
- added REF**: Via-0.6mm, footprints:Via-0.6mm, F.Cu at (132.8, 129.7)
- moved REF** 0.41 mm to (128.9, 129.5)
Routing:
- net Net-(R30-Pad2): track 0.00 -> 161.6 mm, vias 0 -> 1
- net Net-(P3-Pad1): track 0.00 -> 149.0 mm, vias 0 -> 1
- net Net-(C27-Pad1): track 0.00 -> 148.4 mm, vias 0 -> 1
- net Net-(P4-Pad3): track 0.00 -> 107.2 mm, vias 0 -> 1
- net Net-(R38-Pad2): track 0.00 -> 102.3 mm, vias 0 -> 2
- net Net-(P3-Pad3): track 0.00 -> 102.1 mm, vias 0 -> 1
- net Net-(R43-Pad2): track 0.00 -> 93.7 mm, vias 0 -> 2
- net /PI Circuit 2/+5V: track 0.00 -> 93.4 mm, vias 0 -> 1
- net Net-(R10-Pad2): track 68.5 -> 161.2 mm, vias 0 -> 1
- net /PI Circuit 2/set_point_mon: track 0.00 -> 83.2 mm, vias 0 -> 1
- net Net-(R38-Pad1): track 0.00 -> 81.0 mm, vias 0 -> 1
- net /PI Circuit 2/-5V: track 0.00 -> 72.2 mm, vias 0 -> 1
- net Net-(R39-Pad1): track 0.00 -> 71.4 mm, vias 0 -> 2
- net Net-(C34-Pad1): track 0.00 -> 69.9 mm, vias 0 -> 2
- net Net-(R42-Pad1): track 0.00 -> 68.4 mm, vias 0 -> 1
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- added copper zone on B.Cu, net GND
- added copper zone on F.Cu, net GND
Other:
- board text added: "Add gain in parallel. gain=1/(1/33+1/10)=7.7 if switches for 33 and 10 closed"
- board text added: "Dual PI Servo Vutha Labs Shreyas Potnis"
- board text added: "Gain 100 33 10 2 1 0.33 0.1 0"
- board text added: "PI Pole(Hz) 48k 16k 7k 3k 1.6k 700 340 off"
- board text added: "Similarly add PI poles in parallel"
